File: pcb/ShinyAddOn/ShinyAddOn.kicad_pcb (KiCad board)
At the start: 2 copper layers, 50 x 50 mm, 3 parts, among them J1 Conn_02x03_Odd_Even

Commit message: worked on the pcb
Parts:
- added BZ1: Buzzer, Buzzer_Beeper:Buzzer_12x9.5RM7.6, F.Cu at (148.7, 128.5)
- added C1: 1nF, Capacitor_SMD:C_0603_1608Metric_Pad1.08x0.95mm_HandSolder, F.Cu at (150.2, 169.0)
- added C2: 1nF, Capacitor_SMD:C_0603_1608Metric_Pad1.08x0.95mm_HandSolder, F.Cu at (154.8, 169.0)
- added C3: 100nF, Capacitor_SMD:C_0603_1608Metric_Pad1.08x0.95mm_HandSolder, F.Cu at (152.5, 164.8)
- added D10: LED dish bottom left, LED_SMD:LED_0603_1608Metric_Pad1.05x0.95mm_HandSolder, B.Cu at (134.5, 128.5)
- added D11: LED dish bottom right, LED_SMD:LED_0603_1608Metric_Pad1.05x0.95mm_HandSolder, B.Cu at (170.5, 128.5)
- added D12: WS2812B-2020, LED_SMD:LED_WS2812B-2020_PLCC4_2.0x2.0mm, B.Cu at (152.5, 148.2)
- added D2: lower front LED, LED_SMD:LED_0603_1608Metric_Pad1.05x0.95mm_HandSolder, F.Cu at (142.4, 151.5)
- added D3: LED blue right, LED_SMD:LED_0603_1608Metric_Pad1.05x0.95mm_HandSolder, F.Cu at (164.5, 180.5)
- added D4: LED blue left, LED_SMD:LED_0603_1608Metric_Pad1.05x0.95mm_HandSolder, F.Cu at (140.5, 180.5)
- added D5: LED blue front, LED_SMD:LED_0603_1608Metric_Pad1.05x0.95mm_HandSolder, F.Cu at (152.5, 113.2)
- added D6: LED red left, LED_SMD:LED_0603_1608Metric_Pad1.05x0.95mm_HandSolder, F.Cu at (140.5, 161.0)
- added D7: LED red right, LED_SMD:LED_0603_1608Metric_Pad1.05x0.95mm_HandSolder, F.Cu at (164.5, 161.0)
- added D8: LED dish top left, LED_SMD:LED_0603_1608Metric_Pad1.05x0.95mm_HandSolder, F.Cu at (134.5, 128.5)
- added D9: LED dish top right, LED_SMD:LED_0603_1608Metric_Pad1.05x0.95mm_HandSolder, F.Cu at (170.5, 128.5)
- added J3: GPIO, Jumper:SolderJumper-2_P1.3mm_Open_RoundedPad1.0x1.5mm, B.Cu at (158.2, 176.2)
- added J4: saucer connetion, Connector_PinSocket_2.54mm:PinSocket_2x03_P2.54mm_Vertical, F.Cu at (149.9, 150.7)
- added J5: SAO Connector, Connector_PinHeader_2.54mm:PinHeader_2x03_P2.54mm_Vertical, B.Cu at (150.0, 174.7)
- added JP1: Jumper_2_Bridged, Jumper:SolderJumper-2_P1.3mm_Bridged_RoundedPad1.0x1.5mm, B.Cu at (160.8, 176.2)
- added R10: 330, Resistor_SMD:R_0603_1608Metric_Pad0.98x0.95mm_HandSolder, F.Cu at (141.5, 128.0)
- added R11: 330, Resistor_SMD:R_0603_1608Metric_Pad0.98x0.95mm_HandSolder, F.Cu at (163.5, 128.0)
- added R12: 330, Resistor_SMD:R_0603_1608Metric_Pad0.98x0.95mm_HandSolder, F.Cu at (145.0, 120.5)
- added R13: 330, Resistor_SMD:R_0603_1608Metric_Pad0.98x0.95mm_HandSolder, F.Cu at (145.0, 136.5)
- added R14: 47, Resistor_SMD:R_0603_1608Metric_Pad0.98x0.95mm_HandSolder, F.Cu at (157.5, 152.0)
- added R2: 330, Resistor_SMD:R_0603_1608Metric_Pad0.98x0.95mm_HandSolder, F.Cu at (139.2, 151.0)
- added R3: 330, Resistor_SMD:R_0603_1608Metric_Pad0.98x0.95mm_HandSolder, F.Cu at (161.0, 176.2)
- added R4: 330, Resistor_SMD:R_0603_1608Metric_Pad0.98x0.95mm_HandSolder, F.Cu at (144.0, 176.2)
- added R5: 330, Resistor_SMD:R_0603_1608Metric_Pad0.98x0.95mm_HandSolder, F.Cu at (160.0, 120.5)
- added R6: 330, Resistor_SMD:R_0603_1608Metric_Pad0.98x0.95mm_HandSolder, F.Cu at (145.5, 176.2)
- added R7: 330, Resistor_SMD:R_0603_1608Metric_Pad0.98x0.95mm_HandSolder, F.Cu at (159.5, 176.2)
- added R8: 10k, Resistor_SMD:R_0603_1608Metric_Pad0.98x0.95mm_HandSolder, F.Cu at (153.2, 169.0)
- added R9: 10k, Resistor_SMD:R_0603_1608Metric_Pad0.98x0.95mm_HandSolder, F.Cu at (151.8, 169.0)
- added SW1: SW_Push, Button_Switch_SMD:SW_Tactile_SPST_NO_Straight_CK_PTS636Sx25SMTRLFS, F.Cu at (140.5, 171.5)
- added SW2: SW_Push, Button_Switch_SMD:SW_Tactile_SPST_NO_Straight_CK_PTS636Sx25SMTRLFS, F.Cu at (164.5, 171.5)
- added U1: CH32V003FxPx, Package_SO:TSSOP-20_4.4x6.5mm_P0.65mm, F.Cu at (152.5, 159.2)
- D1: value LED -> blue front powerled; footprint LED_SMD:LED_0805_2012Metric_Pad1.15x1.40mm_HandSolder -> LED_SMD:LED_0603_1608Metric_Pad1.05x0.95mm_HandSolder
- R1: value R -> 330; footprint Resistor_SMD:R_0805_2012Metric_Pad1.20x1.40mm_HandSolder -> Resistor_SMD:R_0603_1608Metric_Pad0.98x0.95mm_HandSolder
- moved R1 32.0 mm to (160.0, 136.5), turned to 45 degrees
- moved D1 25.4 mm to (152.5, 136.8), turned to 180 degrees
- moved J1 24.6 mm to (150.0, 142.0)
Connections:
- J1 pad 3: /SDA -> /buzzer
- J1 pad 4: /SCL -> /LED dish top left
- J1 pad 5: /GPIO1 -> /LED dish bottom
- J1 pad 6: /GPIO2 -> /LED dish top right
Routing:
- net /red_gondeln_right: track 0.00 -> 35.9 mm, vias 0 -> 2
- net Net-(JP1-B): track 0.00 -> 34.8 mm, vias 0 -> 1
- net VCC: track 0.00 -> 33.8 mm, vias 0 -> 2
- net /red_gondeln_left: track 0.00 -> 33.6 mm, vias 0 -> 2
- net /blue gondeln left: track 0.00 -> 32.1 mm, vias 0 -> 2
- net /sw2: track 0.00 -> 31.5 mm
- net /blue gondeln right: track 0.00 -> 31.1 mm, vias 0 -> 2
- net /sw1: track 0.00 -> 28.9 mm
- net /SCL: track 0.00 -> 19.2 mm, vias 0 -> 1
- net Net-(D6-A): track 0.00 -> 18.9 mm
- net Net-(D7-A): track 0.00 -> 18.7 mm
- net /SDA: track 0.00 -> 17.6 mm, vias 0 -> 1
- net /LED dish bottom: track 0.00 -> 8.64 mm
- net GND: track 0.00 -> 6.70 mm, vias 1 -> 4
- net Net-(D3-A): track 0.00 -> 6.25 mm
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- removed copper zone on F.Cu, net VCC
Other:
- board size 50 x 50 mm -> 42 x 71.5 mm
- board text added: "NCC-1701-D"
- board text removed: "TOP"

Commit message: pcb updated
Parts:
- removed D12: WS2812B-2020, LED_SMD:LED_WS2812B-2020_PLCC4_2.0x2.0mm
- removed R14: 47, Resistor_SMD:R_0603_1608Metric_Pad0.98x0.95mm_HandSolder
- D2: moved to B.Cu
- J1: value Conn_02x03_Odd_Even -> Conn_02x04_Odd_Even; footprint Connector_PinHeader_2.54mm:PinHeader_2x03_P2.54mm_Vertical -> Connector_PinHeader_2.54mm:PinHeader_2x04_P2.54mm_Vertical
- J4: footprint Connector_PinSocket_2.54mm:PinSocket_2x03_P2.54mm_Vertical -> Connector_PinSocket_2.54mm:PinSocket_2x04_P2.54mm_Vertical
- moved R1 15.0 mm to (145.0, 136.5), turned to 135 degrees
- moved R13 15.0 mm to (160.0, 136.5), turned to 45 degrees
- moved R2 13.5 mm to (152.5, 148.2), turned to 0 degrees
- moved D2 10.6 mm to (152.5, 148.2)
- moved D1 2.25 mm to (152.5, 139.0), turned to 0 degrees
- moved J1 1.28 mm to (148.7, 142.0)
- moved J4 1.22 mm to (148.7, 150.7)
- moved R10 0.50 mm to (141.5, 128.5)
- moved R11 0.50 mm to (163.5, 128.5)
- turned D10 to 90 degrees
- turned R5 to 135 degrees
Connections:
- D10 pad 1: /LED dish bottom -> /LED dish bottom l
- D11 pad 1: /LED dish bottom -> /LED dish bottom r
- J1 pad 5: /LED dish bottom -> /LED dish bottom l
- J4 pad 5: /LED dish bottom -> /LED dish bottom l
- U1 pad 1: /LED dish bottom -> /LED dish bottom l
- U1 pad 2: Net-(U1-PD5) -> /LED dish bottom r
Routing:
- net /blue_front: track 0.00 -> 42.5 mm, vias 0 -> 1
- net /LED dish bottom l: track 0.00 -> 34.9 mm
- net /LED dish bottom r: track 0.00 -> 32.7 mm
- net /buzzer: track 0.00 -> 31.2 mm, vias 0 -> 2
- net VCC: track 33.8 -> 64.3 mm, vias 2 -> 3
- net /LED dish top right: track 3.23 -> 32.1 mm, vias 0 -> 2
- net /LED dish top left: track 5.36 -> 33.5 mm, vias 1 -> 2
- net GND: track 6.70 -> 29.2 mm, vias 4 -> 9
- net Net-(D10-A): track 0.00 -> 17.1 mm, vias 0 -> 1
- net Net-(U1-PD0): track 0.69 -> 16.7 mm, vias 0 -> 2
- net Net-(D11-A): track 0.00 -> 12.5 mm, vias 0 -> 1
- net Net-(D1-A): track 0.00 -> 11.0 mm
- net Net-(D5-A): track 0.00 -> 9.37 mm, vias 0 -> 2
- net /LED dish bottom: track 8.64 -> 0.00 mm
- net Net-(D9-A): track 0.00 -> 7.76 mm, vias 0 -> 2
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- added copper zone on F.Cu, net VCC
Other:
- board size 42 x 71.5 mm -> 41.9 x 71.5 mm
- board text added: "GPIO1-Prog"
- board text added: "USS Enterprise"
- board text added: "https://github.com/dg3vw/Trekkie_Addon"
- board text removed: "GP1"
- board text removed: "GP2"
- board text removed: "VCC"
- board text removed: "gnd"
